File: ICEDevBoard.kicad_pcb (KiCad board)
At the start: 4 copper layers, 100 x 100 mm, 233 parts, among them J101 USB4215-03-A_REVA, J301 program, J401 VGA, J501 Joystick, J502 SJ2-35813B-SMT-TR, J503 Keyboard, J504 Mouse, J505 MSD-1-A, J701 PMOD, Q101 BC847, SW701 SW_Push, SW702 SW_Push, SW703 SW_Push, U101 AP2127K-3.3, U102 AP2127K-2.5, U103 AP2127K-1.2, U201 93LC56BT-I/OT, U202 FT232H, U301 ICE40HX8K-BG121, U302 W25Q32JVSS, U401 ADV7123, U501 SN74LVC8T245PWR, U502 PCM5102A, U503 SN74LV1T34DBV, U601 IS61WV5128EDBLL-10TLI, U701 74AHC595, U702 74AHC595, Y201 12Mhz, Y301 50Mhz, Y302 12Mhz

Commit message: Working on layout
Parts:
- C312: footprint Capacitor_SMD:C_0603_1608Metric -> Capacitor_SMD:C_0805_2012Metric
- C602, L301, L302, R305: moved to B.Cu
- moved L302 65.8 mm to (154.4, 84.5), turned to 180 degrees
- moved L301 64.0 mm to (154.4, 87.2), turned to 180 degrees
- moved TP104 60.3 mm to (166.4, 77.0), turned to 0 degrees
- moved C111 58.3 mm to (169.8, 77.2)
- moved R305 56.0 mm to (152.6, 96.3)
- moved U103 50.4 mm to (164.7, 81.1)
- moved C110 50.4 mm to (161.3, 81.1)
- moved C112 50.4 mm to (170.4, 80.8)
- moved U302 50.1 mm to (120.5, 105.0)
- moved J301 48.7 mm to (131.5, 101.5)
- moved U102 45.2 mm to (164.5, 86.7)
- moved C104 45.2 mm to (161.1, 86.7)
- moved C108 45.2 mm to (170.4, 86.2)
- moved C106 42.9 mm to (169.8, 89.8)
- moved TP102 42.7 mm to (166.0, 89.8), turned to 180 degrees
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Routing:
- net Net-(U301E-VCCPLL0): track 0.00 -> 14.9 mm, vias 0 -> 3
- net GND: track 0.00 -> 7.86 mm, vias 0 -> 5
- net +3V3: track 0.00 -> 5.25 mm, vias 0 -> 5
- net Net-(U301E-VPP_2V5): track 0.00 -> 3.08 mm, vias 0 -> 2
- net unconnected-(U301B-IOR_161-PadB11): track 1.55 -> 2.39 mm
- added copper zone on In2.Cu, net +3V3
Other:
- board text added: "1.2V"
- board text added: "2.5V"
- board text added: "3.3V"
- board text added: "FLASH"
- board text added: "FPGA"
- board text added: "FPGA DONE"
- board text added: "PROG"
- board text added: "VBUS"

Commit message: Initial FPGA layout done
Parts:
- C205, C213, C215, C216, C217, C301, C302, C303, C304, C305, C306, C307, C308, C309, C310, C311, C314, C315, C317, C318: moved to B.Cu
- C312: footprint Capacitor_SMD:C_0805_2012Metric -> Capacitor_SMD:C_0603_1608Metric
- moved C304 74.9 mm to (156.4, 82.3)
- moved C302 70.7 mm to (153.3, 82.3), turned to 180 degrees
- moved C216 41.8 mm to (104.6, 121.2), turned to 180 degrees
- moved C215 37.3 mm to (104.7, 124.6), turned to 180 degrees
- moved C205 33.1 mm to (124.3, 125.2)
- moved C217 32.4 mm to (125.1, 121.8), turned to 180 degrees
- moved C213 31.5 mm to (128.8, 122.5)
- moved C203 31.0 mm to (133.2, 125.3), turned to -90 degrees
- moved C201 27.1 mm to (131.7, 129.3), turned to 180 degrees
- moved C314 23.4 mm to (71.5, 92.1), turned to 180 degrees
- moved C315 21.3 mm to (71.5, 94.5), turned to 180 degrees
- moved C303 16.9 mm to (88.0, 80.3), turned to 180 degrees
- moved C317 16.7 mm to (75.9, 99.1), turned to 180 degrees
- moved C318 16.7 mm to (75.9, 102.1), turned to 180 degrees
- moved C301 14.0 mm to (88.0, 77.3), turned to 180 degrees
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Connections:
- U301 pad A1: unconnected-(U301A-IOT_225-PadA1) -> /FPGA/MEM_A10
- U301 pad A10: unconnected-(U301A-IOT_170-PadA10) -> /FPGA/MOUSE_DATA
- U301 pad A11: unconnected-(U301A-IOT_168-PadA11) -> /FPGA/SD_SELECT
- U301 pad A2: unconnected-(U301A-IOT_222-PadA2) -> /FPGA/MEM_A11
- U301 pad A3: unconnected-(U301A-IOT_223-PadA3) -> /FPGA/PMOD6
- U301 pad A4: unconnected-(U301A-IOT_211-PadA4) -> /FPGA/PMOD1
- U301 pad A5: unconnected-(U301A-IOT_207-PadA5) -> /FPGA/JOY_SEL
- U301 pad A6: unconnected-(U301A-IOT_206-PadA6) -> /FPGA/JOY_D0
- U301 pad A7: unconnected-(U301A-IOT_192-PadA7) -> /FPGA/JOY_D1
- U301 pad A8: unconnected-(U301A-IOT_190-PadA8) -> /FPGA/JOY_D4
- U301 pad A9: unconnected-(U301A-IOT_178-PadA9) -> /FPGA/KBD_CLK
- U301 pad B1: unconnected-(U301D-IOL_2A-PadB1) -> /FPGA/MEM_A13
- U301 pad B11: unconnected-(U301B-IOR_161-PadB11) -> /FPGA/SD_MOSI
- U301 pad B2: unconnected-(U301D-IOL_2B-PadB2) -> /FPGA/MEM_A12
- U301 pad B3: unconnected-(U301A-IOT_221-PadB3) -> /FPGA/PMOD3
- U301 pad B4: unconnected-(U301A-IOT_219-PadB4) -> /FPGA/PMOD5
- U301 pad B5: unconnected-(U301A-IOT_208-PadB5) -> /FPGA/PMOD0
- U301 pad B8: unconnected-(U301A-IOT_177-PadB8) -> /FPGA/JOY_D3
- U301 pad B9: unconnected-(U301A-IOT_174-PadB9) -> /FPGA/KBD_DATA
- U301 pad C1: unconnected-(U301D-IOL_5B-PadC1) -> /FPGA/MEM_D4
- U301 pad C11: unconnected-(U301B-IOR_160-PadC11) -> /FPGA/SD_CLOCK
- U301 pad C2: unconnected-(U301D-IOL_5A-PadC2) -> /FPGA/MEM_A14
- U301 pad C3: unconnected-(U301D-IOL_4B-PadC3) -> /FPGA/PMOD7
- U301 pad C4: unconnected-(U301D-IOL_4A-PadC4) -> /FPGA/PMOD2
- U301 pad C7: unconnected-(U301A-IOT_191-PadC7) -> /FPGA/JOY_D5
- U301 pad C9: unconnected-(U301A-IOT_172-PadC9) -> /FPGA/MOUSE_CLK
- U301 pad D1: unconnected-(U301D-IOL_8B-PadD1) -> /FPGA/MEM_D7
- U301 pad D10: unconnected-(U301B-IOR_154-PadD10) -> /FPGA/SD_MISO
- U301 pad D11: unconnected-(U301B-IOR_152-PadD11) -> /FPGA/SND_BCK
- U301 pad D2: unconnected-(U301D-IOL_9A-PadD2) -> /FPGA/MEM_D5
- U301 pad D3: unconnected-(U301D-IOL_9B-PadD3) -> /FPGA/MEM_D6
- U301 pad D5: unconnected-(U301A-IOT_212-PadD5) -> /FPGA/PMOD4
- U301 pad D7: unconnected-(U301A-IOT_181-PadD7) -> /FPGA/JOY_D2
- U301 pad D9: unconnected-(U301B-IOR_147-PadD9) -> /FPGA/SD_DETECT
- U301 pad E1: unconnected-(U301D-IOL_8A-PadE1) -> /FPGA/MEM_A17
- U301 pad E10: unconnected-(U301B-IOR_141_GBIN2-PadE10) -> /FPGA/SND_LRCK
- U301 pad E11: unconnected-(U301B-IOR_148-PadE11) -> /FPGA/~{VGA_BLANK}
- U301 pad E2: unconnected-(U301D-IOL_10A-PadE2) -> /FPGA/MEM_A15
- U301 pad E3: unconnected-(U301D-IOL_10B-PadE3) -> /FPGA/MEM_A16
- U301 pad E8: unconnected-(U301B-IOR_146-PadE8) -> /FPGA/VGA_R2
- U301 pad E9: unconnected-(U301B-IOR_144-PadE9) -> /FPGA/SND_DIN
- U301 pad F1: unconnected-(U301D-IOL_12A-PadF1) -> /FPGA/MEM_A7
- U301 pad F10: unconnected-(U301B-IOR_136-PadF10) -> /FPGA/VGA_HSYNC
- U301 pad F11: unconnected-(U301B-IOR_140_GBIN3-PadF11) -> /FPGA/VGA_CLOCK
- U301 pad F2: unconnected-(U301D-IOL_12B-PadF2) -> /FPGA/MEM_A9
- U301 pad F3: unconnected-(U301D-IOL_13B_GBIN7-PadF3) -> /FPGA/MEM_A18
- U301 pad F4: unconnected-(U301D-IOL_13A-PadF4) -> /FPGA/MEM_A8
- U301 pad F9: unconnected-(U301B-IOR_137-PadF9) -> /FPGA/VGA_VSYNC
- U301 pad G1: unconnected-(U301D-IOL_14A_GBIN6-PadG1) -> /FPGA/~{SRAM_WE}
- U301 pad G10: unconnected-(U301B-IOR_120-PadG10) -> /FPGA/VGA_R0
- U301 pad G11: unconnected-(U301B-IOR_129-PadG11) -> /FPGA/VGA_R1
- U301 pad G2: unconnected-(U301D-IOL_14B-PadG2) -> /FPGA/MEM_A5
- U301 pad G3: unconnected-(U301D-IOL_17A-PadG3) -> /FPGA/MEM_A6
- U301 pad G8: unconnected-(U301B-IOR_118-PadG8) -> /FPGA/VGA_R3
- U301 pad H1: unconnected-(U301D-IOL_18A-PadH1) -> /FPGA/MEM_D1
- U301 pad H10: unconnected-(U301B-IOR_116-PadH10) -> /FPGA/VGA_B0
- U301 pad H11: unconnected-(U301B-IOR_119-PadH11) -> /FPGA/VGA_R4
- U301 pad H2: unconnected-(U301D-IOL_18B-PadH2) -> /FPGA/MEM_D2
- U301 pad H3: unconnected-(U301D-IOL_17B-PadH3) -> /FPGA/MEM_D3
- U301 pad H7: unconnected-(U301C-IOB_87-PadH7) -> /FPGA/VGA_G3
- U301 pad H9: unconnected-(U301C-IOB_104_CBSEL1-PadH9) -> /FPGA/VGA_B2
- U301 pad J1: unconnected-(U301D-IOL_23A-PadJ1) -> /FPGA/~{SRAM_CE}
- U301 pad J10: unconnected-(U301B-IOR_117-PadJ10) -> /FPGA/VGA_B4
- U301 pad J11: unconnected-(U301B-IOR_114-PadJ11) -> /FPGA/VGA_B1
- U301 pad J2: unconnected-(U301D-IOL_25B-PadJ2) -> /FPGA/MEM_A4
- U301 pad J3: unconnected-(U301C-IOB_57-PadJ3) -> /FPGA/MEM_D0
- U301 pad J4: unconnected-(U301C-IOB_64-PadJ4) -> /FPGA/SEG_CLK
- U301 pad J5: unconnected-(U301C-IOB_78-PadJ5) -> /FPGA/LED3
- U301 pad J7: unconnected-(U301C-IOB_86-PadJ7) -> /FPGA/VGA_G1
- U301 pad J8: unconnected-(U301C-IOB_91-PadJ8) -> /FPGA/VGA_G5
- U301 pad K1: unconnected-(U301D-IOL_23B-PadK1) -> /FPGA/MEM_A3
- U301 pad K11: unconnected-(U301B-IOR_115-PadK11) -> /FPGA/VGA_B3
- U301 pad K2: unconnected-(U301D-IOL_25A-PadK2) -> /FPGA/MEM_A2
- U301 pad K3: unconnected-(U301C-IOB_63-PadK3) -> /FPGA/SEG_DATA
- U301 pad K4: unconnected-(U301C-IOB_73-PadK4) -> /FPGA/LED2
- U301 pad K5: unconnected-(U301C-IOB_79-PadK5) -> /FPGA/BUTTON1
- U301 pad K6: unconnected-(U301C-IOB_82_GBIN4-PadK6) -> /FPGA/BUTTON3
- U301 pad K7: unconnected-(U301C-IOB_89-PadK7) -> /FPGA/VGA_G0
- U301 pad L1: unconnected-(U301C-IOB_56-PadL1) -> /FPGA/MEM_A1
- U301 pad L2: unconnected-(U301C-IOB_61-PadL2) -> /FPGA/MEM_A0
- U301 pad L3: unconnected-(U301C-IOB_71-PadL3) -> /FPGA/SEG_LOAD
- U301 pad L4: unconnected-(U301C-IOB_72-PadL4) -> /FPGA/LED1
- U301 pad L5: unconnected-(U301C-IOB_81_GBIN5-PadL5) -> /FPGA/BUTTON2
- U301 pad L7: unconnected-(U301C-IOB_94-PadL7) -> /FPGA/VGA_G2
- U301 pad L8: unconnected-(U301C-IOB_103_CBSEL0-PadL8) -> /FPGA/VGA_G4
Routing:
- net unconnected-(U301B-IOR_146-PadE8): track 5.11 -> 0.00 mm, vias 1 -> 0
- net /FPGA/VGA_R2: track 0.00 -> 5.11 mm, vias 0 -> 1
- net unconnected-(U301C-IOB_87-PadH7): track 4.33 -> 0.00 mm, vias 1 -> 0
- net /FPGA/VGA_G3: track 0.00 -> 4.33 mm, vias 0 -> 1
- net unconnected-(U301D-IOL_13A-PadF4): track 4.28 -> 0.00 mm, vias 1 -> 0
- net /FPGA/MEM_A8: track 0.00 -> 4.28 mm, vias 0 -> 1
- net unconnected-(U301A-IOT_181-PadD7): track 4.12 -> 0.00 mm, vias 1 -> 0
- net /FPGA/JOY_D2: track 0.00 -> 4.12 mm, vias 0 -> 1
- net unconnected-(U301B-IOR_118-PadG8): track 4.07 -> 0.00 mm
- net /FPGA/VGA_R3: track 0.00 -> 4.07 mm
- net unconnected-(U301A-IOT_212-PadD5): track 4.07 -> 0.00 mm, vias 1 -> 0
- net /FPGA/PMOD4: track 0.00 -> 4.07 mm, vias 0 -> 1
- net unconnected-(U301C-IOB_104_CBSEL1-PadH9): track 3.78 -> 0.00 mm
- net /FPGA/VGA_B2: track 0.00 -> 3.78 mm
- net unconnected-(U301D-IOL_9B-PadD3): track 3.53 -> 0.00 mm, vias 1 -> 0
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Other:
- board text added: "Audio"
- board text added: "BUTTON1"
- board text added: "BUTTON2"
- board text added: "BUTTON3"
- board text added: "Joystick"
- board text added: "Keyboard"
- board text added: "LED1"
- board text added: "LED2"
- board text added: "LED3"
- board text added: "Mouse"
- board text added: "PMOD"
- board text added: "SD Card"
- board text added: "VGA"
