File: ICEDevBoard.kicad_pcb (KiCad board)
At the start: 4 copper layers, 100 x 100 mm, 233 parts, among them J101 USB4215-03-A_REVA, J301 program, J401 VGA, J501 Joystick, J502 SJ2-35813B-SMT-TR, J503 Keyboard, J504 Mouse, J505 MSD-1-A, J701 PMOD, Q101 BC847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

Commit message: Latest changes
Parts:
- added TP105: GND, TestPoint:TestPoint_THTPad_D1.0mm_Drill0.5mm, F.Cu at (138.7, 146.6)
- added TP106: GND, TestPoint:TestPoint_THTPad_D1.0mm_Drill0.5mm, F.Cu at (175.7, 77.5)
- added TP107: GND, TestPoint:TestPoint_THTPad_D1.0mm_Drill0.5mm, F.Cu at (136.7, 72.2)
- added TP108: GND, TestPoint:TestPoint_THTPad_D1.0mm_Drill0.5mm, F.Cu at (104.9, 83.9)
- C301, C303: moved to F.Cu
- moved C311 89.7 mm to (166.9, 71.5), turned to -90 degrees
- moved C317 87.7 mm to (163.1, 89.4)
- moved C315 79.2 mm to (150.2, 85.8), turned to 0 degrees
- moved C314 73.6 mm to (144.7, 85.0), turned to 0 degrees
- moved C308 70.4 mm to (152.7, 95.4), turned to 0 degrees
- moved C306 68.2 mm to (147.4, 89.3)
- moved C301 66.9 mm to (154.4, 85.2), turned to 0 degrees
- moved C303 66.7 mm to (154.4, 86.9), turned to 0 degrees
- moved C309 64.7 mm to (147.3, 91.6)
- moved C305 64.5 mm to (140.8, 79.7), turned to -90 degrees
- moved C307 62.0 mm to (152.7, 93.8), turned to 0 degrees
- moved C310 58.8 mm to (141.2, 95.4)
- moved TP101 52.0 mm to (102.3, 137.4)
- moved C318 41.9 mm to (115.7, 89.0)
- moved C204 12.1 mm to (114.7, 121.2), turned to 0 degrees
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Routing:
- net /FPGA/CDONE: track 56.2 -> 114.7 mm, vias 2 -> 3
- net /FPGA/FTDI_SPICLK: track 38.5 -> 96.3 mm, vias 2 -> 5
- net /FPGA/~{FTDI_SPISS}: track 49.4 -> 102.6 mm, vias 2 -> 4
- net /FPGA/FTDI_MOSI: track 1.95 -> 54.7 mm, vias 0 -> 2
- net /FPGA/FTDI_MISO: track 1.97 -> 53.6 mm, vias 0 -> 1
- net /FPGA/~{CRESET}: track 23.2 -> 64.8 mm, vias 0 -> 2
- net Net-(U701-QE): track 0.00 -> 38.7 mm
- net Net-(U701-QD): track 0.00 -> 29.3 mm
- net Net-(U201-CS): track 0.00 -> 24.1 mm
- net Net-(U701-QC): track 0.00 -> 23.2 mm, vias 0 -> 2
- net +5V: track 199.7 -> 221.9 mm, vias 13 -> 16
- net Net-(U701-QH'): track 0.00 -> 21.8 mm, vias 0 -> 2
- net +2V5: track 14.3 -> 33.0 mm, vias 0 -> 1
- net /USB Programming/VPHY: track 4.63 -> 23.1 mm, vias 0 -> 2
- net GND: track 177.2 -> 194.6 mm, vias 92 -> 106
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Other:
- board text added: "GND"
