File: programming.kicad_sch (KiCad schematic)
At the start: 42 parts, among them U201 93LC56BT-I/OT, U202 FT232H, Y201 12Mhz

Commit message: Working on board layout
Parts:
- D201, D202: footprint LED_SMD:LED_1210_3225Metric -> LED_SMD:LED_1206_3216Metric
- R206, R207: value 0R -> 22R
Changed lines of the file:
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@@
 			)
 		)
-		(property "Value" "0R"
+		(property "Value" "22R"
 			(at 112.014 68.326 90)
 			(effects
@@
 			)
 		)
-		(property "Footprint" "LED_SMD:LED_1210_3225Metric"
+		(property "Footprint" "LED_SMD:LED_1206_3216Metric"
 			(at 271.78 92.71 0)
 			(effects
@@
 			)
 		)
-		(property "Footprint" "LED_SMD:LED_1210_3225Metric"
+		(property "Footprint" "LED_SMD:LED_1206_3216Metric"
 			(at 260.35 92.71 0)
 			(effects
@@
 			)
 		)
-		(property "Value" "0R"
+		(property "Value" "22R"
 			(at 112.014 61.214 90)
 			(effects

Commit message: Reworking layout
Connections:
- net VBUS renamed +5V
